Commit message: First compilation

File: smart_template_description/urdf/smart_template.urdf.xacro (robot description, xacro)
@@ -1,15 +1,21 @@
 <?xml version="1.0"?>
 <robot xmlns:xacro="http://wiki.ros.org/xacro" name="$(arg name)">
+  <!-- ros2_control URDF -->
+  <xacro:include filename="$(find smart_template_description)/urdf/smart_template.ros2_control.xacro"/>
   <!-- Argument for needle_type -->
   <xacro:arg name="needle_type" default="default"/>
   <xacro:arg name="zframe_config" default="default"/>
+  <xacro:arg name="robot_mode" default="default"/>
   <!-- smart_template URDF -->
-  <xacro:include filename="$(find smart_template_cpp)/description/urdf/smart_template.xacro"/>
-  <xacro:smart_template needle_type="$(arg needle_type)">
+  <xacro:include filename="$(find smart_template_description)/urdf/smart_template.xacro"/>
+  <xacro:smart_template needle_type="$(arg needle_type)" robot_mode="$(arg robot_mode)">
   </xacro:smart_template>
   <!-- zFrame URDF -->
-  <xacro:include filename="$(find smart_template_cpp)/description/urdf/zframe.xacro"/>
+  <xacro:include filename="$(find smart_template_description)/urdf/zframe.xacro"/>
   <xacro:zframe zframe_config="$(arg zframe_config)">
   </xacro:zframe>
+  <!-- ros2_control URDF -->
+  <xacro:smart_template_ros2_control>
+  </xacro:smart_template_ros2_control>
   <!-- create link fixed to the "world" -->
   <link name="world" />

File: smart_template_description/urdf/smart_template.xacro (robot description, xacro)
@@ -1,5 +1,5 @@
 <?xml version="1.0"?>
 <robot xmlns:xacro="http://wiki.ros.org/xacro">
-  <xacro:macro name="smart_template" params="needle_type">
+  <xacro:macro name="smart_template" params="robot_mode needle_type">
     <!-- Define limit values for each needle type -->
     <xacro:property name="insertion_upper_limit" value="0.115"/>
@@ -17,8 +17,5 @@
     </xacro:if>
     <!-- Include materials -->
-    <xacro:include filename="$(find smart_template_cpp)/description/urdf/materials.xacro" />
-    <!-- Include ros2_control -->
-    <xacro:include filename="$(find smart_template_cpp)/description/urdf/smart_template.ros2_control.xacro" />
-    <xacro:smart_template_ros2_control/>
+    <xacro:include filename="$(find smart_template_description)/urdf/materials.xacro" />
     <!-- Define Links -->
     <link name="base_link">
@@ -26,5 +23,5 @@
         <origin xyz="0 0 0" rpy="0 0 ${-pi/2}"/>
         <geometry>
-          <mesh filename="package://smart_template_cpp/description/meshes/base_link.stl"/>
+          <mesh filename="package://smart_template_description/meshes/base_link.stl"/>
         </geometry>
         <material name="silver"/>
@@ -35,5 +32,5 @@
         <origin xyz="0 0 0" rpy="0 0 ${-pi/2}"/>
         <geometry>
-          <mesh filename="package://smart_template_cpp/description/meshes/vertical_link.stl"/>
+          <mesh filename="package://smart_template_description/meshes/vertical_link.stl"/>
         </geometry>
         <material name="silver"/>
@@ -44,5 +41,5 @@
         <origin xyz="0 0 0" rpy="0 0 ${-pi/2}"/>
         <geometry>
-          <mesh filename="package://smart_template_cpp/description/meshes/horizontal_link.stl"/>
+          <mesh filename="package://smart_template_description/meshes/horizontal_link.stl"/>
         </geometry>
         <material name="silver"/>
@@ -53,5 +50,5 @@
         <origin xyz="0 0 0" rpy="0 0 ${-pi/2}"/>
         <geometry>
-          <mesh filename="package://smart_template_cpp/description/meshes/needle_link_${needle_type}.stl"/>
+          <mesh filename="package://smart_template_description/meshes/needle_link_${needle_type}.stl"/>
         </geometry>
         <material name="silver"/>
@@ -64,5 +61,14 @@
       <child link="vertical_link"/>
       <axis xyz="0.0 0.0 1.0"/>
-      <limit upper="0.025" lower="-0.025" effort="100" velocity="100"/>
+      <!-- conditional limits -->
+      <xacro:if value="$(eval robot_mode == 'calibration')">
+        <limit upper="1e6" lower="-1e6" effort="100" velocity="1e6"/>
+      </xacro:if>
+      <xacro:unless value="$(eval robot_mode == 'calibration')">
+        <limit upper="0.025" lower="-0.025" effort="100" velocity="100"/>
+      </xacro:unless>
+      <!-- custom extension -->
+      <channel>C</channel>
+      <mm_to_count>1430.0</mm_to_count>
     </joint>
     <joint name="horizontal_joint" type="prismatic">
@@ -71,5 +77,14 @@
       <child link="horizontal_link"/>
       <axis xyz="1.0 0.0 0.0"/>
-      <limit upper="0.03" lower="-0.03" effort="100" velocity="100"/>
+      <!-- conditional limits -->
+      <xacro:if value="$(eval robot_mode == 'calibration')">
+        <limit upper="1e6" lower="-1e6" effort="100" velocity="1e6"/>
+      </xacro:if>
+      <xacro:unless value="$(eval robot_mode == 'calibration')">
+        <limit upper="0.03" lower="-0.03" effort="100" velocity="100"/>
+      </xacro:unless>
+      <!-- custom extension -->
+      <channel>A</channel>
+      <mm_to_count>715.0</mm_to_count>
     </joint>
     <joint name="insertion_joint" type="prismatic">
@@ -78,5 +93,14 @@
       <child link="needle_link"/>
       <axis xyz="0.0 1.0 0.0"/>
-      <limit upper="${insertion_upper_limit}" lower="0.0" effort="100" velocity="100"/>
+      <!-- conditional limits -->
+      <xacro:if value="$(eval robot_mode == 'calibration')">
+        <limit upper="1e6" lower="-1e6" effort="100" velocity="1e6"/>
+      </xacro:if>
+      <xacro:unless value="$(eval robot_mode == 'calibration')">
+        <limit upper="${insertion_upper_limit}" lower="0.0" effort="100" velocity="100"/>
+      </xacro:unless>
+      <!-- custom extension -->
+      <channel>B</channel>
+      <mm_to_count>-1574.8031</mm_to_count>
     </joint>
   </xacro:macro>

Commit message: included world frame tf static broadcaster in robot launch

File: smart_template_description/urdf/smart_template.urdf.xacro (robot description, xacro)
@@ -18,10 +18,3 @@
   <xacro:smart_template_ros2_control  sim_level="$(arg sim_level)">
   </xacro:smart_template_ros2_control>
-  <!-- create link fixed to the "world" -->
-  <link name="world" />
-  <joint name="base_joint" type="fixed">
-    <origin xyz="0 0 0" rpy="0 0 0"/>
-    <parent link="world"/>
-    <child link="base_link" />
-  </joint>
 </robot>
