Commit message: Working with ros2_control

File: smart_template_description/urdf/smart_template.ros2_control.xacro (robot description, xacro)
@@ -1,8 +1,13 @@
 <?xml version="1.0"?>
 <robot xmlns:xacro="http://www.ros.org/wiki/xacro">
-  <xacro:macro name="smart_template_ros2_control">
+  <xacro:macro name="smart_template_ros2_control" params="sim_level">
     <ros2_control name="smart_template" type="system">
       <hardware>
-        <plugin>galil_driver/GalilSystemHardwareInterface</plugin>
+        <xacro:if value="${int(sim_level) == 1}">
+          <plugin>mock_components/GenericSystem</plugin>
+        </xacro:if>
+        <xacro:if value="${int(sim_level) == 2}">
+          <plugin>galil_driver/GalilSystemHardwareInterface</plugin>
+        </xacro:if>
       </hardware>
       <joint name="insertion_joint">

File: smart_template_description/urdf/smart_template.urdf.xacro (robot description, xacro)
@@ -1,10 +1,9 @@
 <?xml version="1.0"?>
 <robot xmlns:xacro="http://wiki.ros.org/xacro" name="$(arg name)">
-  <!-- ros2_control URDF -->
-  <xacro:include filename="$(find smart_template_description)/urdf/smart_template.ros2_control.xacro"/>
-  <!-- Argument for needle_type -->
+  <!-- Arguments -->
+  <xacro:arg name="sim_level" default="1"/>
+  <xacro:arg name="robot_mode" default="default"/>
   <xacro:arg name="needle_type" default="default"/>
   <xacro:arg name="zframe_config" default="default"/>
-  <xacro:arg name="robot_mode" default="default"/>
   <!-- smart_template URDF -->
   <xacro:include filename="$(find smart_template_description)/urdf/smart_template.xacro"/>
@@ -16,5 +15,6 @@
   </xacro:zframe>
   <!-- ros2_control URDF -->
-  <xacro:smart_template_ros2_control>
+  <xacro:include filename="$(find smart_template_description)/urdf/smart_template.ros2_control.xacro"/>
+  <xacro:smart_template_ros2_control  sim_level="$(arg sim_level)">
   </xacro:smart_template_ros2_control>
   <!-- create link fixed to the "world" -->

Commit message: Zframe new registration. Launch with position_controller only

File: smart_template_description/urdf/smart_template.ros2_control.xacro (robot description, xacro)
@@ -11,4 +11,18 @@
         </xacro:if>
       </hardware>
+      <joint name="horizontal_joint">
+        <command_interface name="position">
+          <param name="min">-0.03</param>
+          <param name="max"> 0.03</param>
+        </command_interface>
+        <command_interface name="velocity">
+          <param name="min">-0.005</param>
+          <param name="max"> 0.005</param>
+        </command_interface>
+        <state_interface name="position">
+          <param name="initial_value">0</param>
+        </state_interface>
+        <state_interface name="velocity"/>
+      </joint>
       <joint name="insertion_joint">
         <command_interface name="position">
@@ -25,22 +39,8 @@
         <state_interface name="velocity"/>
       </joint>
-      <joint name="horizontal_joint">
-        <command_interface name="position">
-          <param name="min">-0.03</param>
-          <param name="max"> 0.03</param>
-        </command_interface>
-        <command_interface name="velocity">
-          <param name="min">-0.005</param>
-          <param name="max"> 0.005</param>
-        </command_interface>
-        <state_interface name="position">
-          <param name="initial_value">0</param>
-        </state_interface>
-        <state_interface name="velocity"/>
-      </joint>
       <joint name="vertical_joint">
         <command_interface name="position">
-          <param name="min">   0</param>
-          <param name="max">0.05</param>
+          <param name="min">-0.025</param>
+          <param name="max">0.025</param>
         </command_interface>
         <command_interface name="velocity">

File: smart_template_description/urdf/zframe.xacro (robot description, xacro)
@@ -8,7 +8,11 @@
       <xacro:property name="zframe_position" value="0.0 0.0980 -0.1283"/> <!-- Position (x, y, z) -->
     </xacro:if>
-    <xacro:if value="${zframe_config == 'new'}">  <!-- zframe from registration experiment in AMIGO (2025-04-24)-->
+    <xacro:if value="${zframe_config == 'test'}">  <!-- zframe from registration experiment in AMIGO (2025-04-24)-->
       <xacro:property name="zframe_orientation" value="-0.9990810696561544 -0.022101423357745315 0.03672187349962075 -0.020810007551375062 0.9991641103988661 0.035185134034339226 -0.037468819763572525 0.03438861763171322 -0.9987059378014156"/> <!-- Rotation matrix (row by row) -->
       <xacro:property name="zframe_position" value="0.001171932293919652 0.10549880638836385 -0.11120061509823658"/> <!-- Position (x, y, z) -->
+    </xacro:if>
+    <xacro:if value="${zframe_config == 'new'}">  <!-- zframe from registration experiment in AMIGO (2025-07-23)-->
+      <xacro:property name="zframe_orientation" value="-0.9996147025670941 0.014578846766073413 0.023618849514765904 0.01389168105492629 0.9994828181328841 -0.029001386987696023 -0.024029440919981136 -0.028662061839630798 -0.9993002853456078"/> <!-- Rotation matrix (row by row) -->
+      <xacro:property name="zframe_position" value="0.004914398868714972 0.10075025081155526 -0.11873539242196507"/> <!-- Position (x, y, z) -->
     </xacro:if>
     <xacro:if value="${zframe_config == 'old'}"> <!-- zframe from SmartNeedle Animal Experiment in 221 Longwood (2023-12-20) -->

Commit message: Moveit package

File: smart_template_description/urdf/smart_template.ros2_control.xacro (robot description, xacro)
@@ -1,11 +1,38 @@
 <?xml version="1.0"?>
 <robot xmlns:xacro="http://www.ros.org/wiki/xacro">
-  <xacro:macro name="smart_template_ros2_control" params="sim_level">
+  <xacro:macro name="smart_template_ros2_control" params="use_mock_hardware robot_mode needle_type">
+    <!-- Match URDF joint limit logic -->
+    <xacro:property name="horizontal_min" value="-0.03"/>
+    <xacro:property name="horizontal_max" value="0.03"/>
+    <xacro:property name="vertical_min" value="-0.025"/>
+    <xacro:property name="vertical_max" value="0.025"/>
+    <xacro:property name="insertion_min" value="0.0"/>
+    <xacro:property name="insertion_max" value="0.115"/>
+    <xacro:if value="${needle_type == 'default'}">
+      <xacro:property name="insertion_max" value="0.115"/>
+    </xacro:if>
+    <xacro:if value="${needle_type == 'stylet'}">
+      <xacro:property name="insertion_max" value="0.115"/>
+    </xacro:if>
+    <xacro:if value="${needle_type == 'smartneedle'}">
+      <xacro:property name="insertion_max" value="0.165"/>
+    </xacro:if>
+    <xacro:if value="${needle_type == 'biopsygun'}">
+      <xacro:property name="insertion_max" value="0.175"/>
+    </xacro:if>
+    <xacro:if value="${robot_mode == 'calibration'}">
+      <xacro:property name="horizontal_min" value="-1000000.0"/>
+      <xacro:property name="horizontal_max" value="1000000.0"/>
+      <xacro:property name="vertical_min" value="-1000000.0"/>
+      <xacro:property name="vertical_max" value="1000000.0"/>
+      <xacro:property name="insertion_min" value="-1000000.0"/>
+      <xacro:property name="insertion_max" value="1000000.0"/>
+    </xacro:if>
     <ros2_control name="smart_template" type="system">
       <hardware>
-        <xacro:if value="${int(sim_level) == 1}">
+        <xacro:if value="${use_mock_hardware}">
           <plugin>mock_components/GenericSystem</plugin>
         </xacro:if>
-        <xacro:if value="${int(sim_level) == 2}">
+        <xacro:if value="${not use_mock_hardware}">
           <plugin>galil_driver/GalilSystemHardwareInterface</plugin>
         </xacro:if>
@@ -13,10 +40,10 @@
       <joint name="horizontal_joint">
         <command_interface name="position">
-          <param name="min">-0.03</param>
-          <param name="max"> 0.03</param>
+          <param name="min">${horizontal_min}</param>
+          <param name="max">${horizontal_max}</param>
         </command_interface>
         <command_interface name="velocity">
           <param name="min">-0.005</param>
-          <param name="max"> 0.005</param>
+          <param name="max">0.005</param>
         </command_interface>
         <state_interface name="position">
@@ -27,10 +54,10 @@
       <joint name="insertion_joint">
         <command_interface name="position">
-          <param name="min">0</param>
-          <param name="max">0.1</param>
+          <param name="min">${insertion_min}</param>
+          <param name="max">${insertion_max}</param>
         </command_interface>
         <command_interface name="velocity">
           <param name="min">-0.005</param>
-          <param name="max"> 0.005</param>
+          <param name="max">0.005</param>
         </command_interface>
         <state_interface name="position">
@@ -41,10 +68,10 @@
       <joint name="vertical_joint">
         <command_interface name="position">
-          <param name="min">-0.025</param>
-          <param name="max">0.025</param>
+          <param name="min">${vertical_min}</param>
+          <param name="max">${vertical_max}</param>
         </command_interface>
         <command_interface name="velocity">
           <param name="min">-0.005</param>
-          <param name="max"> 0.005</param>
+          <param name="max">0.005</param>
         </command_interface>
         <state_interface name="position">

File: smart_template_description/urdf/smart_template.urdf.xacro (robot description, xacro)
@@ -2,5 +2,5 @@
 <robot xmlns:xacro="http://wiki.ros.org/xacro" name="$(arg name)">
   <!-- Arguments -->
-  <xacro:arg name="sim_level" default="1"/>
+  <xacro:arg name="use_mock_hardware" default="true"/>
   <xacro:arg name="robot_mode" default="default"/>
   <xacro:arg name="needle_type" default="default"/>
@@ -16,5 +16,5 @@
   <!-- ros2_control URDF -->
   <xacro:include filename="$(find smart_template_description)/urdf/smart_template.ros2_control.xacro"/>
-  <xacro:smart_template_ros2_control  sim_level="$(arg sim_level)">
+  <xacro:smart_template_ros2_control use_mock_hardware="$(arg use_mock_hardware)" robot_mode="$(arg robot_mode)" needle_type="$(arg needle_type)">
   </xacro:smart_template_ros2_control>
 </robot>

File: smart_template_description/urdf/smart_template.xacro (robot description, xacro)
@@ -27,4 +27,10 @@
         <material name="silver"/>
       </visual>
+      <collision>
+        <origin xyz="0 0 0" rpy="0 0 ${-pi/2}"/>
+          <geometry>
+            <mesh filename="package://smart_template_description/meshes/base_link.stl"/>
+          </geometry>
+      </collision>
     </link>
     <link name="vertical_link">
@@ -36,4 +42,10 @@
         <material name="silver"/>
       </visual>
+      <collision>
+        <origin xyz="0 0 0" rpy="0 0 ${-pi/2}"/>
+        <geometry>
+          <mesh filename="package://smart_template_description/meshes/vertical_link.stl"/>
+        </geometry>
+      </collision>
     </link>
     <link name="horizontal_link">
@@ -45,4 +57,10 @@
         <material name="silver"/>
       </visual>
+      <collision>
+        <origin xyz="0 0 0" rpy="0 0 ${-pi/2}"/>
+        <geometry>
+          <mesh filename="package://smart_template_description/meshes/horizontal_link.stl"/>
+        </geometry>
+      </collision>
     </link>
     <link name="needle_link">
@@ -54,4 +72,10 @@
         <material name="silver"/>
       </visual>
+      <collision>
+        <origin xyz="0 0 0" rpy="0 0 ${-pi/2}"/>
+        <geometry>
+          <mesh filename="package://smart_template_description/meshes/needle_link_${needle_type}.stl"/>
+        </geometry>
+      </collision>
     </link>
     <!-- Define joints -->
